Commit message: fix joints names

File: src/cobot630pro_moveit_config/cobot630pro_moveit_config/config/firefighter.ros2_control.xacro (robot description, xacro)
@@ -8,43 +8,43 @@
                 <plugin>mock_components/GenericSystem</plugin>
             </hardware>
-            <joint name="joint1_to_base">
+            <joint name="joint0">
                 <command_interface name="position"/>
                 <state_interface name="position">
-                  <param name="initial_value">${initial_positions['joint1_to_base']}</param>
+                  <param name="initial_value">${initial_positions['joint0']}</param>
                 </state_interface>
                 <state_interface name="velocity"/>
             </joint>
-            <joint name="joint2_to_joint1">
+            <joint name="joint1">
                 <command_interface name="position"/>
                 <state_interface name="position">
-                  <param name="initial_value">${initial_positions['joint2_to_joint1']}</param>
+                  <param name="initial_value">${initial_positions['joint1']}</param>
                 </state_interface>
                 <state_interface name="velocity"/>
             </joint>
-            <joint name="joint3_to_joint2">
+            <joint name="joint2">
                 <command_interface name="position"/>
                 <state_interface name="position">
-                  <param name="initial_value">${initial_positions['joint3_to_joint2']}</param>
+                  <param name="initial_value">${initial_positions['joint2']}</param>
                 </state_interface>
                 <state_interface name="velocity"/>
             </joint>
-            <joint name="joint4_to_joint3">
+            <joint name="joint3">
                 <command_interface name="position"/>
                 <state_interface name="position">
-                  <param name="initial_value">${initial_positions['joint4_to_joint3']}</param>
+                  <param name="initial_value">${initial_positions['joint3']}</param>
                 </state_interface>
                 <state_interface name="velocity"/>
             </joint>
-            <joint name="joint5_to_joint4">
+            <joint name="joint4">
                 <command_interface name="position"/>
                 <state_interface name="position">
-                  <param name="initial_value">${initial_positions['joint5_to_joint4']}</param>
+                  <param name="initial_value">${initial_positions['joint4']}</param>
                 </state_interface>
                 <state_interface name="velocity"/>
             </joint>
-            <joint name="joint6_to_joint5">
+            <joint name="joint5">
                 <command_interface name="position"/>
                 <state_interface name="position">
-                  <param name="initial_value">${initial_positions['joint6_to_joint5']}</param>
+                  <param name="initial_value">${initial_positions['joint5']}</param>
                 </state_interface>
                 <state_interface name="velocity"/>

File: src/mycobot630pro_description/urdf/mycobot_pro_630/mycobot_pro_630.urdf (robot description, URDF)
Before this commit: robot firefighter, 7 links, 6 joints
Joints:
- removed joint joint1_to_base
- removed joint joint2_to_joint1
- removed joint joint3_to_joint2
- removed joint joint4_to_joint3
- removed joint joint5_to_joint4
- removed joint joint6_to_joint5
- added joint joint0: type revolute, parent base, child link1, origin xyz=0 0 0.22934 rpy=0 0 0, axis 0 0 1, limit lower=-3.14 upper=3.14159 effort=1000.0 velocity=0
- added joint joint1: type revolute, parent link1, child link2, origin xyz=0 0  0 rpy=1.5707 0 0, axis 0 0 -1, limit lower=-4.71 upper=1.5707 effort=1000.0 velocity=0
- added joint joint2: type revolute, parent link2, child link3, origin xyz=0.27 0 0    rpy=0 0 0, axis  0 0 -1, limit lower=-2.61 upper=2.618 effort=1000.0 velocity=0
- added joint joint3: type revolute, parent link3, child link4, origin xyz=0.267 0  -0.0745 rpy=0 0 0, axis  0 0 -1, limit lower=-4.53 upper=1.3962 effort=1000.0 velocity=0
- added joint joint4: type revolute, parent link4, child link5, origin xyz=0 -0.095 0.002 rpy=1.5707 -1.5707 0, axis 0 0 1, limit lower=-2.93 upper=2.9321 effort=1000.0 velocity=0
- added joint joint5: type revolute, parent link5, child link6, origin xyz=-0.054 0 0 rpy=-1.5707 0 0 , axis -1 0 0, limit lower=-3.03 upper=3.0368 effort=1000.0 velocity=0
